File: TAH BOARD VER 4.0/TAH BOARD VER 4.0.sch (EAGLE design)
At the start: 33 parts, among them J1 AVR_SPI_PRG, U1 ATMEGA32U4, U2 3.3V_REG_LDOSMD

Commit message: TAH Shields new version update
Changed lines of the file:
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@@
 <?xml version="1.0" encoding="utf-8"?>
 <!DOCTYPE eagle SYSTEM "eagle.dtd">
-<eagle version="6.4">
+<eagle version="7.0.0">
 <drawing>
 <settings>
@@
 <layer number="54" name="bGND_GNDA" color="1" fill="9" visible="no" active="no"/>
 <layer number="56" name="wert" color="7" fill="1" visible="no" active="no"/>
+<layer number="57" name="tCAD" color="7" fill="1" visible="no" active="no"/>
 <layer number="91" name="Nets" color="2" fill="1" visible="yes" active="yes"/>
 <layer number="92" name="Busses" color="1" fill="1" visible="yes" active="yes"/>
@@
 <layer number="132" name="bAdjust" color="7" fill="1" visible="no" active="yes"/>
 <layer number="144" name="Drill_legend" color="7" fill="1" visible="yes" active="yes"/>
+<layer number="150" name="Notes" color="7" fill="1" visible="no" active="yes"/>
 <layer number="151" name="HeatSink" color="7" fill="1" visible="yes" active="yes"/>
 <layer number="152" name="_bDocu" color="7" fill="1" visible="yes" active="yes"/>
+<layer number="153" name="FabDoc1" color="6" fill="1" visible="no" active="no"/>
+<layer number="154" name="FabDoc2" color="2" fill="1" visible="no" active="no"/>
+<layer number="155" name="FabDoc3" color="7" fill="15" visible="no" active="no"/>
 <layer number="199" name="Contour" color="7" fill="1" visible="yes" active="yes"/>
 <layer number="200" name="200bmp" color="1" fill="10" visible="yes" active="yes"/>
@@
 </instance>
 <instance part="GND5" gate="1" x="102.87" y="33.02"/>
-<instance part="5V" gate="G$1" x="102.87" y="63.5"/>
+<instance part="5V" gate="G$1" x="102.87" y="62.23"/>
 <instance part="GND7" gate="1" x="130.81" y="20.32"/>
 <instance part="P+3" gate="G$1" x="52.07" y="195.58"/>
@@
 <wire x1="115.57" y1="40.64" x2="115.57" y2="45.72" width="0.1524" layer="91"/>
 <wire x1="110.49" y1="58.42" x2="115.57" y2="58.42" width="0.1524" layer="91"/>
+<junction x="115.57" y="40.64"/>
+<junction x="115.57" y="58.42"/>
 </segment>
 <segment>
@@
 <net name="5V" class="0">
 <segment>
-<wire x1="102.87" y1="63.5" x2="102.87" y2="60.96" width="0.1524" layer="91"/>
+<wire x1="102.87" y1="62.23" x2="102.87" y2="60.96" width="0.1524" layer="91"/>
 <wire x1="102.87" y1="60.96" x2="102.87" y2="58.42" width="0.1524" layer="91"/>
 <wire x1="95.25" y1="60.96" x2="102.87" y2="60.96" width="0.1524" layer="91"/>
@@
 <wire x1="217.17" y1="100.33" x2="223.52" y2="100.33" width="0.1524" layer="91"/>
 <label x="223.52" y="100.33" size="1.778" layer="95" rot="R180"/>
+<junction x="217.17" y="100.33"/>
 </segment>
 </net>
@@
 <pinref part="JP5" gate="G$1" pin="6"/>
 <wire x1="217.17" y1="97.79" x2="223.52" y2="97.79" width="0.1524" layer="91"/>
+<junction x="217.17" y="97.79"/>
 </segment>
 </net>
@@
 <pinref part="JP5" gate="G$1" pin="5"/>
 <wire x1="217.17" y1="95.25" x2="223.52" y2="95.25" width="0.1524" layer="91"/>
+<junction x="217.17" y="95.25"/>
 </segment>
 </net>
@@
 <pinref part="JP5" gate="G$1" pin="4"/>
 <wire x1="217.17" y1="92.71" x2="223.52" y2="92.71" width="0.1524" layer="91"/>
+<junction x="217.17" y="92.71"/>
 </segment>
 </net>
@@
 <pinref part="JP5" gate="G$1" pin="3"/>
 <wire x1="217.17" y1="90.17" x2="223.52" y2="90.17" width="0.1524" layer="91"/>
+<junction x="217.17" y="90.17"/>
 </segment>
 </net>
@@
 <pinref part="JP5" gate="G$1" pin="2"/>
 <wire x1="217.17" y1="87.63" x2="223.52" y2="87.63" width="0.1524" layer="91"/>
+<junction x="217.17" y="87.63"/>
 </segment>
 </net>
@@
 <pinref part="JP5" gate="G$1" pin="1"/>
 <wire x1="217.17" y1="85.09" x2="223.52" y2="85.09" width="0.1524" layer="91"/>
+<junction x="217.17" y="85.09"/>
 </segment>
 </net>
@@
 <pinref part="C2" gate="G$1" pin="2"/>
 <wire x1="123.19" y1="55.88" x2="123.19" y2="58.42" width="0.1524" layer="91"/>
+<junction x="123.19" y="55.88"/>
 </segment>
 </net>
@@
 <pinref part="C3" gate="G$1" pin="2"/>
 <wire x1="123.19" y1="40.64" x2="123.19" y2="45.72" width="0.1524" layer="91"/>
+<junction x="123.19" y="45.72"/>
 </segment>
 </net>
@@
 </sheet>
 </sheets>
+<errors>
+</errors>
 </schematic>
 </drawing>
