File: Tah Board Ver 1.0/Tah Board Ver 1.0.sch (EAGLE design)
At the start: 33 parts, among them J1 AVR_SPI_PRG, U1 ATMEGA32U4, U2 3.3V_REG_LDOSMD

Commit message: Added latest design files
Parts:
- removed JP1: M12PTH, SparkFun-Connectors:M12PTH
- removed JP4, JP5: (no value), SparkFun-Connectors:M07
- removed TP1, TP2, TP3, TP4: TPTP11SQ, testpad:TPTP11SQ
- added JP6, JP7: M13, SparkFun-Connectors:M13
- added R5, R6: 1k, SparkFun-Resistors:RESISTOR1206
- U1: device FTDI modifed:ATMEGA32U4TQFP -> SparkFun-DigitalIC:ATMEGA32U4QFN
Connections:
- new net N$4: BLE.2, R5.1
- new net N$5: BLE.4, R6.1
- net 3.3V: now also JP6.11; no longer JP1.4
- net 5V: now also JP6.10, JP6.7; no longer JP1.3, JP5.7
- net A0: now also JP6.6; no longer JP5.6
- net A1: now also JP6.5; no longer JP5.5
- net A2: now also JP6.4; no longer JP5.4
- net A3: now also JP6.3; no longer JP5.3
- net A4: now also JP6.2; no longer JP5.2
- net A5: now also JP6.1; no longer JP5.1
- net D+: no longer TP2.TP
- net D-: no longer TP1.TP
- net D10: now also JP7.11; no longer JP1.9
- net D11: now also JP7.12; no longer JP1.8
- net D12: now also JP7.13; no longer JP1.7
- net D13: now also JP6.13; no longer JP1.6
- net D2: now also JP7.3; no longer JP4.3
- net D3: now also JP7.4; no longer JP4.4
- net D4: now also JP7.5; no longer JP4.5
- net D5: now also JP7.6; no longer JP4.6
- net D6: now also JP7.7; no longer JP4.7
- net D7: now also JP7.8; no longer JP1.12
- net D8: now also JP7.9; no longer JP1.11
- net D9: now also JP7.10; no longer JP1.10
- net GND: now also JP6.8, JP6.9; no longer JP1.1, JP1.2, TP3.TP
- net RST: now also JP6.12; no longer JP1.5
- net RX: now also JP7.2, R6.2; no longer BLE.4, JP4.2
- net TX: now also JP7.1, R5.2; no longer BLE.2, JP4.1
- net VBUS: no longer TP4.TP
Other:
- note added: "Designed By: Dhiraj Jadhao"
- note added: "Tah is an open source development board that helps you create your own projects that can connect to your smart phone"
- note added: "http://tah.io"
- moved on the sheet: C4, C5, C6, C7, C8, C9, J1, L, R7, R9, STATUS, U2

Commit message: Updated production ready files for Tah and shields
Parts:
- L: value Yellow -> Green
- ON: value Green -> Red
- U1: device SparkFun-DigitalIC:ATMEGA32U4QFN -> SparkFun-Retired:ATMEGA32U4QFN2
- renumbered STATUS to B
Changed lines of the file:
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@@
 <setting verticaltext="up"/>
 </settings>
-<grid distance="0.1" unitdist="inch" unit="inch" style="lines" multiple="1" display="yes" altdistance="0.01" altunitdist="inch" altunit="inch"/>
+<grid distance="0.1" unitdist="inch" unit="inch" style="lines" multiple="1" display="no" altdistance="0.01" altunitdist="inch" altunit="inch"/>
 <layers>
-<layer number="1" name="Top" color="4" fill="1" visible="no" active="no"/>
-<layer number="16" name="Bottom" color="1" fill="1" visible="no" active="no"/>
-<layer number="17" name="Pads" color="2" fill="1" visible="no" active="no"/>
-<layer number="18" name="Vias" color="2" fill="1" visible="no" active="no"/>
-<layer number="19" name="Unrouted" color="6" fill="1" visible="no" active="no"/>
-<layer number="20" name="Dimension" color="15" fill="1" visible="no" active="no"/>
-<layer number="21" name="tPlace" color="16" fill="1" visible="no" active="no"/>
-<layer number="22" name="bPlace" color="7" fill="1" visible="no" active="no"/>
-<layer number="23" name="tOrigins" color="15" fill="1" visible="no" active="no"/>
-<layer number="24" name="bOrigins" color="15" fill="1" visible="no" active="no"/>
-<layer number="25" name="tNames" color="7" fill="1" visible="no" active="no"/>
-<layer number="26" name="bNames" color="7" fill="1" visible="no" active="no"/>
-<layer number="27" name="tValues" color="7" fill="1" visible="no" active="no"/>
-<layer number="28" name="bValues" color="7" fill="1" visible="no" active="no"/>
+<layer number="1" name="Top" color="4" fill="1" visible="yes" active="no"/>
+<layer number="16" name="Bottom" color="1" fill="1" visible="yes" active="no"/>
+<layer number="17" name="Pads" color="2" fill="1" visible="yes" active="no"/>
+<layer number="18" name="Vias" color="2" fill="1" visible="yes" active="no"/>
+<layer number="19" name="Unrouted" color="6" fill="1" visible="yes" active="no"/>
+<layer number="20" name="Dimension" color="15" fill="1" visible="yes" active="no"/>
+<layer number="21" name="tPlace" color="7" fill="1" visible="yes" active="no"/>
+<layer number="22" name="bPlace" color="7" fill="1" visible="yes" active="no"/>
+<layer number="23" name="tOrigins" color="15" fill="1" visible="yes" active="no"/>
+<layer number="24" name="bOrigins" color="15" fill="1" visible="yes" active="no"/>
+<layer number="25" name="tNames" color="7" fill="1" visible="yes" active="no"/>
+<layer number="26" name="bNames" color="7" fill="1" visible="yes" active="no"/>
+<layer number="27" name="tValues" color="7" fill="1" visible="yes" active="no"/>
+<layer number="28" name="bValues" color="7" fill="1" visible="yes" active="no"/>
 <layer number="29" name="tStop" color="7" fill="3" visible="no" active="no"/>
 <layer number="30" name="bStop" color="7" fill="6" visible="no" active="no"/>
@@
 <layer number="35" name="tGlue" color="7" fill="4" visible="no" active="no"/>
 <layer number="36" name="bGlue" color="7" fill="5" visible="no" active="no"/>
-<layer number="37" name="tTest" color="7" fill="1" visible="no" active="no"/>
-<layer number="38" name="bTest" color="7" fill="1" visible="no" active="no"/>
+<layer number="37" name="tTest" color="7" fill="1" visible="yes" active="no"/>
+<layer number="38" name="bTest" color="7" fill="1" visible="yes" active="no"/>
 <layer number="39" name="tKeepout" color="4" fill="11" visible="no" active="no"/>
 <layer number="40" name="bKeepout" color="1" fill="11" visible="no" active="no"/>
@@
 <layer number="44" name="Drills" color="7" fill="1" visible="no" active="no"/>
 <layer number="45" name="Holes" color="7" fill="1" visible="no" active="no"/>
-<layer number="46" name="Milling" color="3" fill="1" visible="no" active="no"/>
-<layer number="47" name="Measures" color="7" fill="1" visible="no" active="no"/>
-<layer number="48" name="Document" color="7" fill="1" visible="no" active="no"/>
-<layer number="49" name="Reference" color="7" fill="1" visible="no" active="no"/>
-<layer number="50" name="dxf" color="7" fill="1" visible="no" active="no"/>
-<layer number="51" name="tDocu" color="14" fill="1" visible="no" active="no"/>
-<layer number="52" name="bDocu" color="7" fill="1" visible="no" active="no"/>
-<layer number="53" name="tGND_GNDA" color="7" fill="9" visible="no" active="no"/>
-<layer number="54" name="bGND_GNDA" color="1" fill="9" visible="no" active="no"/>
-<layer number="56" name="wert" color="7" fill="1" visible="no" active="no"/>
-<layer number="57" name="tCAD" color="7" fill="1" visible="no" active="no"/>
+<layer number="46" name="Milling" color="3" fill="1" visible="yes" active="no"/>
+<layer number="47" name="Measures" color="7" fill="1" visible="yes" active="no"/>
+<layer number="48" name="Document" color="7" fill="1" visible="yes" active="no"/>
+<layer number="49" name="Reference" color="7" fill="1" visible="yes" active="no"/>
+<layer number="50" name="dxf" color="7" fill="1" visible="yes" active="no"/>
+<layer number="51" name="tDocu" color="7" fill="1" visible="yes" active="no"/>
+<layer number="52" name="bDocu" color="7" fill="1" visible="yes" active="no"/>
+<layer number="53" name="tGND_GNDA" color="7" fill="9" visible="yes" active="no"/>
+<layer number="54" name="bGND_GNDA" color="1" fill="9" visible="yes" active="no"/>
+<layer number="56" name="wert" color="7" fill="1" visible="yes" active="no"/>
+<layer number="57" name="tCAD" color="7" fill="1" visible="yes" active="no"/>
 <layer number="91" name="Nets" color="2" fill="1" visible="yes" active="yes"/>
 <layer number="92" name="Busses" color="1" fill="1" visible="yes" active="yes"/>
@@
 </classes>
 <parts>
-<part name="U1" library="SparkFun-DigitalIC" deviceset="ATMEGA32U4" device="QFN" value="ATMEGA32U4"/>
+<part name="U1" library="SparkFun-Retired" deviceset="ATMEGA32U4" device="QFN2" value="ATMEGA32U4"/>
 <part name="R1" library="SparkFun-Resistors" deviceset="RESISTOR" device="1206" value="10k"/>
 <part name="GND1" library="SparkFun" deviceset="GND" device=""/>
@@
 <part name="R3" library="SparkFun-Resistors" deviceset="RESISTOR" device="1206" value="22"/>
 <part name="R4" library="SparkFun-Resistors" deviceset="RESISTOR" device="1206" value="1k"/>
-<part name="ON" library="1n4148 diode sot 23" deviceset="LED" device="SMT1206" value="Green"/>
+<part name="ON" library="1n4148 diode sot 23" deviceset="LED" device="SMT1206" value="Red"/>
 <part name="GND5" library="SparkFun" deviceset="GND" device=""/>
 <part name="5V" library="SparkFun" deviceset="5V" device=""/>
@@
 <part name="GND14" library="SparkFun" deviceset="GND" device=""/>
 <part name="R7" library="SparkFun-Resistors" deviceset="RESISTOR" device="1206" value="1k"/>
-<part name="L" library="1n4148 diode sot 23" deviceset="LED" device="SMT1206" value="Yellow"/>
+<part name="L" library="1n4148 diode sot 23" deviceset="LED" device="SMT1206" value="Green"/>
 <part name="GND16" library="SparkFun" deviceset="GND" device=""/>
-<part name="STATUS" library="1n4148 diode sot 23" deviceset="LED" device="SMT1206" value="Blue"/>
+<part name="B" library="1n4148 diode sot 23" deviceset="LED" device="SMT1206" value="Blue"/>
 <part name="R9" library="SparkFun-Resistors" deviceset="RESISTOR" device="1206" value="470"/>
 <part name="GND18" library="SparkFun" deviceset="GND" device=""/>
@@
 <instance part="L" gate="G$1" x="209.55" y="71.12"/>
 <instance part="GND16" gate="1" x="209.55" y="58.42"/>
-<instance part="STATUS" gate="G$1" x="135.89" y="185.42"/>
+<instance part="B" gate="G$1" x="135.89" y="185.42"/>
 <instance part="R9" gate="G$1" x="135.89" y="196.85" smashed="yes" rot="R270">
 <attribute name="NAME" x="132.0546" y="198.882" size="1.778" layer="95" rot="R270"/>
@@
 <segment>
 <pinref part="GND18" gate="1" pin="GND"/>
-<pinref part="STATUS" gate="G$1" pin="C"/>
+<pinref part="B" gate="G$1" pin="C"/>
 <wire x1="135.89" y1="173.99" x2="135.89" y2="180.34" width="0.1524" layer="91"/>
 </segment>
@@
 <net name="N$11" class="0">
 <segment>
-<pinref part="STATUS" gate="G$1" pin="A"/>
+<pinref part="B" gate="G$1" pin="A"/>
 <pinref part="R9" gate="G$1" pin="2"/>
 <wire x1="135.89" y1="187.96" x2="135.89" y2="191.77" width="0.1524" layer="91"/>
